Commit message: emergency stop, lasers, ros2 laser scan merger integration. custom 3 wheeled robot hardware and simulation

File: rosbot_description/urdf/common/ros2_control.urdf.xacro (robot description, xacro)
@@ -30,25 +30,14 @@
         <param name="connection_timeout_ms">30000</param>
         <param name="connection_check_period_ms">1000</param>
-        <!-- order of velocity commands to be published in motors_cmd Float32MultiArray msg -->
         <param name="velocity_command_joint_order">
-          rr_wheel_joint, rl_wheel_joint, fr_wheel_joint, fl_wheel_joint
+          left_wheel_joint, right_wheel_joint
         </param>
       </hardware>
-      <joint name="fl_wheel_joint">
+      <joint name="left_wheel_joint">
         <command_interface name="velocity" />
         <state_interface name="position" />
         <state_interface name="velocity" />
       </joint>
-      <joint name="fr_wheel_joint">
-        <command_interface name="velocity" />
-        <state_interface name="position" />
-        <state_interface name="velocity" />
-      </joint>
-      <joint name="rl_wheel_joint">
-        <command_interface name="velocity" />
-        <state_interface name="position" />
-        <state_interface name="velocity" />
-      </joint>
-      <joint name="rr_wheel_joint">
+      <joint name="right_wheel_joint">
         <command_interface name="velocity" />
         <state_interface name="position" />
@@ -61,25 +50,14 @@
     <ros2_control name="${ns}${name}" type="system">
       <hardware>
-        <plugin>gz_ros2_control/GazeboSimSystem</plugin>
-        <!-- <xacro:if value="${simulation_engine == 'webots'}">
-          <plugin>webots_ros2_control::Ros2ControlSystem</plugin>
-        </xacro:if> -->
+        <!-- <plugin>gz_ros2_control/GazeboSimSystem</plugin> -->
+        <plugin>rosbot_gazebo/EStopSystem</plugin>
+        <param name="e_stop_initial_state">true</param>
       </hardware>
-      <joint name="fl_wheel_joint">
+      <joint name="left_wheel_joint">
         <command_interface name="velocity" />
         <state_interface name="position" />
         <state_interface name="velocity" />
       </joint>
-      <joint name="fr_wheel_joint">
-        <command_interface name="velocity" />
-        <state_interface name="position" />
-        <state_interface name="velocity" />
-      </joint>
-      <joint name="rl_wheel_joint">
-        <command_interface name="velocity" />
-        <state_interface name="position" />
-        <state_interface name="velocity" />
-      </joint>
-      <joint name="rr_wheel_joint">
+      <joint name="right_wheel_joint">
         <command_interface name="velocity" />
         <state_interface name="position" />

File: rosbot_description/urdf/rosbot.urdf.xacro (robot description, xacro)
@@ -6,4 +6,10 @@
   <xacro:arg name="namespace" default="" />
   <xacro:arg name="use_sim" default="false" />
+  <xacro:arg name="xyz1" default="0 0 0" />
+  <xacro:arg name="rpy1" default="0 0 0" />
+  <xacro:arg name="prefix1" default="front" />
+  <xacro:arg name="xyz2" default="0 0 0" />
+  <xacro:arg name="rpy2" default="0 0 3.141" />
+  <xacro:arg name="prefix2" default="rear" />
   <xacro:include filename="$(find rosbot_description)/urdf/rosbot/rosbot_macro.urdf.xacro" ns="husarion" />
   <xacro:include filename="$(find husarion_components_description)/urdf/components.urdf.xacro" ns="components" />
@@ -12,5 +18,12 @@
     mecanum="$(arg mecanum)"
     namespace="$(arg namespace)"
-    use_sim="$(arg use_sim)" />
+    use_sim="$(arg use_sim)"
+    xyz1="$(arg xyz1)"
+    rpy1="$(arg rpy1)"
+    prefix1="$(arg prefix1)"
+    xyz2="$(arg xyz2)"
+    rpy2="$(arg rpy2)"
+    prefix2="$(arg prefix2)"
+  />
   <xacro:components.create_components
     components_config_path="$(arg components_config)"

File: rosbot_description/urdf/rosbot/body.urdf.xacro (robot description, xacro)
@@ -2,5 +2,5 @@
 <robot xmlns:xacro="http://www.ros.org/wiki/xacro">
   <!-- body defining macro -->
-  <xacro:macro name="body" params="wheel_radius namespace">
+  <xacro:macro name="body" params="wheel_radius namespace xyz1 rpy1 prefix1 xyz2 rpy2 prefix2">
     <xacro:include filename="$(find rosbot_description)/urdf/rosbot/components/vl53lox.urdf.xacro" ns="range_sensor" />
     <link name="base_link" />
@@ -13,7 +13,10 @@
       <visual>
         <geometry>
-          <mesh filename="package://rosbot_description/meshes/rosbot/body.stl" scale="0.001 0.001 0.001" />
+          <mesh filename="package://rosbot_description/meshes/rosbot/panda_body.stl" scale="0.001 0.001 0.001" />
         </geometry>
-        <origin xyz="0.0 0.0 -0.0173" rpy="${pi/2} 0.0 ${pi/2}" />
+        <!-- <geometry>
+          <box size="0.221 0.103 0.09" />
+        </geometry> -->
+        <origin xyz="-0.02761 0.0 0.0114" rpy="3.141 0.0 0.0" />
         <material name="Black">
           <color rgba="0.1 0.1 0.1 1.0" />
@@ -25,37 +28,18 @@
       <collision>
         <geometry>
-          <box size="0.197 0.150 0.080" />
+          <box size="0.221 0.103 0.09036" />
         </geometry>
-        <origin xyz="0.0 0.0 ${0.040 - 0.02}" rpy="0.0 0.0 0.0" />
+        <origin xyz="-0.02434 0 0.02922" rpy="0.0 0.0 0.0" />
       </collision>
       <inertial>
-        <mass value="1.728" />
-        <inertia ixx="0.004162" ixy="0.0"     ixz="0.0"
-                                iyy="0.00651" iyz="0.0"
-                                              izz="0.008828" />
-        <origin xyz="0.0 0.0 ${0.040 - 0.02}" rpy="0.0 0.0 0.0" />
+        <mass value="0.916" />
+        <inertia ixx="0.001019" ixy="0.000062"     ixz="-0.000127"
+                                iyy="0.003027"        iyz="-0.000029"
+                                              izz="0.003307" />
+        <origin xyz="-0.02706 0.00089 0.03205" rpy="0.0 0.0 0.0" />
       </inertial>
     </link>
-    <joint name="body_to_cover_joint" type="fixed">
-      <origin xyz="0.0 0.0 0.0603" rpy="0.0 0.0 0.0" />
-      <parent link="body_link" />
-      <child link="cover_link" />
-    </joint>
-    <link name="cover_link">
-      <visual>
-        <geometry>
-          <mesh filename="package://rosbot_description/meshes/rosbot/cover.stl" scale="0.001 0.001 0.001" />
-        </geometry>
-        <origin xyz="0.0 0.0 -0.002" rpy="${pi/2} 0.0 ${pi/2}" />
-        <material name="Black">
-          <color rgba="0.1 0.1 0.1 1.0" />
-        </material>
-        <gazebo reference="cover_link">
-          <material>Gazebo/Black</material>
-        </gazebo>
-      </visual>
-    </link>
     <joint name="body_to_imu_joint" type="fixed">
-      <origin xyz="0.003 -0.0495 0.04332" rpy="0.0 0.0 0.0" />
+      <origin xyz="0.02258 0.02495 0.07329" rpy="0.0 0.0 0.0" />
       <parent link="body_link" />
       <child link="imu_link" />
@@ -63,13 +47,11 @@
     <link name="imu_link" />
     <joint name="body_to_camera_joint" type="fixed">
-      <origin xyz="-0.0141 0.0 0.125" rpy="0.0 0.0 0.0" />
+      <origin xyz="0.06087 0.0 0.10240" rpy="0.0 0.0 0.0" />
       <parent link="body_link" />
       <child link="camera_mount_link" />
     </joint>
     <link name="camera_mount_link" />
-    <xacro:range_sensor.vl53lox parent="body_link" xyz="0.0926  0.05 0.015"   rpy="0.0 0.0 ${radians(12.5)}"  prefix="fl" namespace="${namespace}" />
-    <xacro:range_sensor.vl53lox parent="body_link" xyz="0.0926 -0.05 0.015"   rpy="0.0 0.0 ${radians(-12.5)}" prefix="fr" namespace="${namespace}" />
-    <xacro:range_sensor.vl53lox parent="body_link" xyz="-0.0926 0.05 0.0115"  rpy="0.0 0.0 ${radians(167.5)}" prefix="rl" namespace="${namespace}" />
-    <xacro:range_sensor.vl53lox parent="body_link" xyz="-0.0926 -0.05 0.0115" rpy="0.0 0.0 ${radians(192.5)}" prefix="rr" namespace="${namespace}" />
+    <xacro:range_sensor.vl53lox parent="body_link" xyz="${xyz1}"   rpy="${rpy1}"  prefix="${prefix1}" namespace="${namespace}" />
+    <xacro:range_sensor.vl53lox parent="body_link" xyz="${xyz2}"   rpy="${rpy2}"  prefix="${prefix2}" namespace="${namespace}" />
   </xacro:macro>
 </robot>

File: rosbot_description/urdf/rosbot/components/vl53lox.urdf.xacro (robot description, xacro)
@@ -14,29 +14,31 @@
     <gazebo reference="${prefix}_range">
       <sensor name="${ns}${prefix}_range" type='gpu_lidar'>
-        <topic>${ns}range/${prefix}</topic>
+        <topic>/${ns}_range_${prefix}</topic>
         <gz_frame_id>${prefix}_range</gz_frame_id>
-        <update_rate>5.0</update_rate>
-        <ray>
+        <visualize>true</visualize>
+        <!-- <update_rate>0.518</update_rate> -->
+        <update_rate>10</update_rate>
+        <lidar>
           <scan>
             <horizontal>
-              <samples>1</samples>
+              <samples>46</samples>
               <resolution>1</resolution>
-              <min_angle>-0.01</min_angle>
-              <max_angle>0.01</max_angle>
+              <min_angle>-1.57</min_angle>
+              <max_angle>1.57</max_angle>
             </horizontal>
           </scan>
           <range>
-            <min>0.01</min>
-            <max>0.90</max>
-            <resolution>0.02</resolution>
+            <min>0.03</min>
+            <max>1.2</max>
+            <resolution>0.001</resolution>
           </range>
           <noise>
             <type>gaussian</type>
-            <mean>0.1</mean>
-            <stddev>0.005</stddev>
+            <mean>0</mean>
+            <stddev>0.03</stddev>
           </noise>
-        </ray>
+        </lidar>
         <always_on>true</always_on>
-        <visualize>false</visualize>
+        <visualize>true</visualize>
       </sensor>
     </gazebo>

File: rosbot_description/urdf/rosbot/rosbot_macro.urdf.xacro (robot description, xacro)
@@ -5,20 +5,27 @@
             mecanum
             namespace
-            use_sim">
+            use_sim
+            xyz1
+            rpy1
+            prefix1
+            xyz2
+            rpy2
+            prefix2">
     <!-- PROPERTIES -->
-    <xacro:property name="wheel_radius" value="${0.047 if mecanum else 0.0425}" />
+    <xacro:property name="wheel_radius" value="${0.047 if mecanum else 0.0344}" />
     <!-- INCLUDE ROBOT MACRO -->
     <xacro:include filename="$(find rosbot_description)/urdf/common/gazebo.urdf.xacro" ns="gazebo" />
     <xacro:include filename="$(find rosbot_description)/urdf/common/ros2_control.urdf.xacro" ns="ros2_control" />
     <!-- <xacro:include filename="$(find rosbot_description)/urdf/common/webots.urdf.xacro" ns="webots" /> -->
-    <xacro:include filename="$(find rosbot_description)/urdf/rosbot/body.urdf.xacro" ns="body" />
+    <xacro:include filename="$(find rosbot_description)/urdf/rosbot/body.urdf.xacro" ns="body" />`
     <xacro:include filename="$(find rosbot_description)/urdf/rosbot/wheel.urdf.xacro" ns="wheel" />
     <!-- BODY -->
-    <xacro:body.body wheel_radius="${wheel_radius}" namespace="${namespace}" />
+    <xacro:body.body wheel_radius="${wheel_radius}" namespace="${namespace}" xyz1="${xyz1}" rpy1="${rpy1}" prefix1="${prefix1}" xyz2="${xyz2}" rpy2="${rpy2}" prefix2="${prefix2}" />
     <!-- WHEEL -->
-    <xacro:wheel.wheel wheel_radius="${wheel_radius}" side="fl" mecanum="${mecanum}" />
-    <xacro:wheel.wheel wheel_radius="${wheel_radius}" side="fr" mecanum="${mecanum}" />
-    <xacro:wheel.wheel wheel_radius="${wheel_radius}" side="rl" mecanum="${mecanum}" />
-    <xacro:wheel.wheel wheel_radius="${wheel_radius}" side="rr" mecanum="${mecanum}" />
+    <xacro:wheel.wheel wheel_radius="${wheel_radius}" side="left" mecanum="${mecanum}" />
+    <xacro:wheel.wheel wheel_radius="${wheel_radius}" side="right" mecanum="${mecanum}" />
+    <xacro:unless value="${mecanum}">
+      <xacro:wheel.wheel wheel_radius="${wheel_radius}" side="castor" mecanum="${mecanum}" />
+    </xacro:unless>
     <!-- HARDWARE PLUGINS -->
     <xacro:unless value="${use_sim}">
