Commit message: emergency stop, lasers, ros2 laser scan merger integration. custom 3 wheeled robot hardware and simulation

File: rosbot_description/urdf/rosbot/wheel.urdf.xacro (robot description, xacro)
@@ -3,111 +3,171 @@
   <!-- wheel defining macro -->
   <xacro:macro name="wheel" params="mecanum side wheel_radius">
-    <xacro:property name="wheel_separation_x" value="0.106" />
-    <xacro:if value="${mecanum}">
-      <xacro:property name="wheel_file" value="mecanum" />
-      <xacro:property name="wheel_thickness" value="0.0455" />
-      <xacro:property name="mass" value="0.153" />
-      <xacro:property name="ixx" value="0.000111" />
-      <xacro:property name="iyy" value="0.000169" />
-      <xacro:property name="izz" value="0.000111" />
-      <xacro:property name="wheel_separation_y" value="0.205" />
+    <xacro:unless value="${side == 'castor'}">
+      <xacro:property name="wheel_separation_x" value="0.106" />
+      <xacro:if value="${mecanum}">
+        <xacro:property name="wheel_file" value="mecanum" />
+        <xacro:property name="wheel_thickness" value="0.0455" />
+        <xacro:property name="mass" value="0.153" />
+        <xacro:property name="ixx" value="0.000111" />
+        <xacro:property name="iyy" value="0.000169" />
+        <xacro:property name="izz" value="0.000111" />
+        <xacro:property name="wheel_separation_y" value="0.205" />
+      </xacro:if>
+      <xacro:unless value="${mecanum}">
+        <xacro:property name="wheel_file" value="wheel" />
+        <xacro:property name="wheel_thickness" value="0.025" />
+        <xacro:property name="mass" value="0.035" />
+        <xacro:property name="ixx" value="0.000014" />
+        <xacro:property name="iyy" value="0.000024" />
+        <xacro:property name="izz" value="0.000014" />
+        <xacro:property name="wheel_separation_y" value="0.133" />
+      </xacro:unless>
+      <xacro:if value="${side == 'fl'}">
+        <xacro:property name="x" value="${wheel_separation_x/2.0}" />
+        <xacro:property name="y" value="${wheel_separation_y/2.0}" />
+        <xacro:property name="mesh" value="package://rosbot_description/meshes/rosbot/${wheel_file}_b.dae" />
+        <xacro:property name="scale" value="1.0 1.0 1.0" />
+        <xacro:property name="origin" value="0.0 0.0 0.0" />
+        <xacro:property name="visual_rotation" value="${pi}" />
+        <xacro:property name="fdir" value="1.0 -1.0 0.0" />
+      </xacro:if>
+      <xacro:if value="${side == 'fr'}">
+        <xacro:property name="x" value="${wheel_separation_x/2.0}" />
+        <xacro:property name="y" value="${-wheel_separation_y/2.0}" />
+        <xacro:property name="mesh" value="package://rosbot_description/meshes/rosbot/${wheel_file}_a.dae" />
+        <xacro:property name="scale" value="1.0 1.0 1.0" />
+        <xacro:property name="origin" value="0.0 0.0 0.0" />
+        <xacro:property name="visual_rotation" value="${pi}" />
+        <xacro:property name="fdir" value="1.0 1.0 0.0" />
+      </xacro:if>
+      <xacro:if value="${side == 'rl'}">
+        <xacro:property name="x" value="${-wheel_separation_x/2.0}" />
+        <xacro:property name="y" value="${wheel_separation_y/2.0}" />
+        <xacro:property name="mesh" value="package://rosbot_description/meshes/rosbot/${wheel_file}_a.dae" />
+        <xacro:property name="scale" value="1.0 1.0 1.0" />
+        <xacro:property name="origin" value="0.0 0.0 0.0" />
+        <xacro:property name="visual_rotation" value="${0.0}" />
+        <xacro:property name="fdir" value="1.0 1.0 0.0" />
+      </xacro:if>
+      <xacro:if value="${side == 'rr'}">
+        <xacro:property name="x" value="${-wheel_separation_x/2.0}" />
+        <xacro:property name="y" value="${-wheel_separation_y/2.0}" />
+        <xacro:property name="mesh" value="package://rosbot_description/meshes/rosbot/${wheel_file}_b.dae" />
+        <xacro:property name="scale" value="1.0 1.0 1.0" />
+        <xacro:property name="origin" value="0.0 0.0 0.0" />
+        <xacro:property name="visual_rotation" value="${0.0}" />
+        <xacro:property name="fdir" value="1.0 -1.0 0.0" />
+      </xacro:if>
+      <xacro:if value="${side == 'left'}">
+        <xacro:property name="x" value="0.0" />
+        <xacro:property name="y" value="${wheel_separation_y/2.0}" />
+        <xacro:property name="mesh" value="package://rosbot_description/meshes/rosbot/panda_wheel.stl" />
+        <xacro:property name="scale" value="0.001 0.001 0.001" />
+        <xacro:property name="origin" value="0.00019 -0.07115 -0.01715" />
+        <xacro:property name="visual_rotation" value="${3.141}" />
+        <xacro:property name="fdir" value="1.0 1.0 0.0" />
+      </xacro:if>
+      <xacro:if value="${side == 'right'}">
+        <xacro:property name="x" value="0.0" />
+        <xacro:property name="y" value="${-wheel_separation_y/2.0}" />
+        <xacro:property name="mesh" value="package://rosbot_description/meshes/rosbot/panda_wheel.stl" />
+        <xacro:property name="scale" value="0.001 0.001 0.001" />
+        <xacro:property name="origin" value="0.00019 0.07115 -0.01715" />
+        <xacro:property name="visual_rotation" value="${0.0}" />
+        <xacro:property name="fdir" value="1.0 -1.0 0.0" />
+      </xacro:if>
+      <joint name="${side}_wheel_joint" type="continuous">
+        <parent link="body_link" />
+        <child link="${side}_wheel_link" />
+        <origin xyz="${x} ${y} 0.0" rpy="0.0 0.0 0.0" />
+        <axis xyz="0.0 1.0 0.0" />
+        <limit effort="1.5" velocity="24.0" />
+        <dynamics damping="0.001" friction="0.001" />
+      </joint>
+      <link name="${side}_wheel_link">
+        <visual>
+          <geometry>
+            <mesh filename="${mesh}" scale="${scale}" />
+          </geometry>
+          <origin xyz="${origin}" rpy="0.0 0.0 ${visual_rotation}" />
+        </visual>
+        <collision>
+          <geometry>
+            <cylinder radius="${wheel_radius}" length="${wheel_thickness}" />
+          </geometry>
+          <origin xyz="0.0 0.0 0.0" rpy="${pi/2} 0.0 0.0" />
+        </collision>
+        <inertial>
+          <mass value="${mass}" />
+          <inertia ixx="${ixx}" ixy="0.0"    ixz="0.0"
+                                iyy="${iyy}" iyz="0.0"
+                                            izz="${izz}" />
+        </inertial>
+      </link>
+      <gazebo reference="${side}_wheel_link" xmlns:gz="http://gazeborobotics.org/schema">
+        <xacro:unless value="${mecanum}">
+          <collision>
+            <surface>
+              <friction>
+                <ode>
+                  <mu>1</mu>
+                  <mu2>1</mu2>
+                  <slip1>0.035</slip1>
+                  <slip2>0</slip2>
+                  <fdir1>0 0 1</fdir1>
+                </ode>
+              </friction>
+            </surface>
+          </collision>
+        </xacro:unless>
+        <xacro:if value="${mecanum}">
+          <collision>
+            <surface>
+              <friction>
+                <ode>
+                  <mu>0.8</mu>
+                  <mu2>0.2</mu2>
+                    <slip1>0.035</slip1>
+                  <slip2>0</slip2>
+                  <fdir1 gz:expressed_in="base_link">${fdir}</fdir1>
+                </ode>
+              </friction>
+            </surface>
+          </collision>
+        </xacro:if>
+      </gazebo>
+    </xacro:unless>
+    <xacro:if value="${side == 'castor'}">
+      <xacro:property name="z_offset" value="-0.0219" />
+      <joint name="${side}_wheel_joint" type="fixed">
+        <parent link="body_link"/>
+        <child link="${side}_wheel_link"/>
+        <origin xyz="-0.13176 0.0 ${z_offset}" rpy="0.0 0.0 0.0"/>
+      </joint>
+      <link name="${side}_wheel_link">
+        <visual>
+          <geometry>
+            <sphere radius="0.0125"/> </geometry>
+          <material name="Black"/>
+        </visual>
+        <collision>
+          <geometry>
+            <sphere radius="0.0125"/>
+          </geometry>
+        </collision>
+        <inertial>
+          <mass value="0.037"/>
+          <inertia ixx="0.000008" ixy="0.0"       ixz="0.0"
+                                  iyy="0.000008"  iyz="0.0"
+                                                  izz="0.000008"/>
+        </inertial>
+      </link>
+      <gazebo reference="${side}_wheel_link">
+        <mu1 value="0.001"/> <mu2 value="0.001"/>
+        <kp value="1000000.0"/>
+        <kd value="10.0"/>
+        <material>Gazebo/Black</material>
+      </gazebo>
     </xacro:if>
-    <xacro:unless value="${mecanum}">
-      <xacro:property name="wheel_file" value="wheel" />
-      <xacro:property name="wheel_thickness" value="0.036" />
-      <xacro:property name="mass" value="0.074" />
-      <xacro:property name="ixx" value="0.000041" />
-      <xacro:property name="iyy" value="0.000067" />
-      <xacro:property name="izz" value="0.000041" />
-      <xacro:property name="wheel_separation_y" value="0.192" />
-    </xacro:unless>
-    <xacro:if value="${side == 'fl'}">
-      <xacro:property name="x" value="${wheel_separation_x/2.0}" />
-      <xacro:property name="y" value="${wheel_separation_y/2.0}" />
-      <xacro:property name="mesh" value="package://rosbot_description/meshes/rosbot/${wheel_file}_b.dae" />
-      <xacro:property name="visual_rotation" value="${pi}" />
-      <xacro:property name="fdir" value="1.0 -1.0 0.0" />
-    </xacro:if>
-    <xacro:if value="${side == 'fr'}">
-      <xacro:property name="x" value="${wheel_separation_x/2.0}" />
-      <xacro:property name="y" value="${-wheel_separation_y/2.0}" />
-      <xacro:property name="mesh" value="package://rosbot_description/meshes/rosbot/${wheel_file}_a.dae" />
-      <xacro:property name="visual_rotation" value="${pi}" />
-      <xacro:property name="fdir" value="1.0 1.0 0.0" />
-    </xacro:if>
-    <xacro:if value="${side == 'rl'}">
-      <xacro:property name="x" value="${-wheel_separation_x/2.0}" />
-      <xacro:property name="y" value="${wheel_separation_y/2.0}" />
-      <xacro:property name="mesh" value="package://rosbot_description/meshes/rosbot/${wheel_file}_a.dae" />
-      <xacro:property name="visual_rotation" value="${0.0}" />
-      <xacro:property name="fdir" value="1.0 1.0 0.0" />
-    </xacro:if>
-    <xacro:if value="${side == 'rr'}">
-      <xacro:property name="x" value="${-wheel_separation_x/2.0}" />
-      <xacro:property name="y" value="${-wheel_separation_y/2.0}" />
-      <xacro:property name="mesh" value="package://rosbot_description/meshes/rosbot/${wheel_file}_b.dae" />
-      <xacro:property name="visual_rotation" value="${0.0}" />
-      <xacro:property name="fdir" value="1.0 -1.0 0.0" />
-    </xacro:if>
-    <joint name="${side}_wheel_joint" type="continuous">
-      <parent link="body_link" />
-      <child link="${side}_wheel_link" />
-      <origin xyz="${x} ${y} 0.0" rpy="0.0 0.0 0.0" />
-      <axis xyz="0.0 1.0 0.0" />
-      <limit effort="1.5" velocity="24.0" />
-      <dynamics damping="0.001" friction="0.001" />
-    </joint>
-    <link name="${side}_wheel_link">
-      <visual>
-        <geometry>
-          <mesh filename="${mesh}" scale="1.0 1.0 1.0" />
-        </geometry>
-        <origin xyz="0.0 0.0 0.0" rpy="0.0 0.0 ${visual_rotation}" />
-      </visual>
-      <collision>
-        <geometry>
-          <cylinder radius="${wheel_radius}" length="${wheel_thickness}" />
-        </geometry>
-        <origin xyz="0.0 0.0 0.0" rpy="${pi/2} 0.0 0.0" />
-      </collision>
-      <inertial>
-        <mass value="${mass}" />
-        <inertia ixx="${ixx}" ixy="0.0"    ixz="0.0"
-                              iyy="${iyy}" iyz="0.0"
-                                           izz="${izz}" />
-      </inertial>
-    </link>
-    <gazebo reference="${side}_wheel_link" xmlns:gz="http://gazeborobotics.org/schema">
-      <xacro:unless value="${mecanum}">
-        <collision>
-          <surface>
-            <friction>
-              <ode>
-                <mu>1</mu>
-                <mu2>1</mu2>
-                <slip1>0.035</slip1>
-                <slip2>0</slip2>
-                <fdir1>0 0 1</fdir1>
-              </ode>
-            </friction>
-          </surface>
-        </collision>
-      </xacro:unless>
-      <xacro:if value="${mecanum}">
-        <collision>
-          <surface>
-            <friction>
-              <ode>
-                <mu>0.8</mu>
-                <mu2>0.2</mu2>
-                  <slip1>0.035</slip1>
-                <slip2>0</slip2>
-                <fdir1 gz:expressed_in="base_link">${fdir}</fdir1>
-              </ode>
-            </friction>
-          </surface>
-        </collision>
-      </xacro:if>
-    </gazebo>
   </xacro:macro>
 </robot>
